File: soulmeasurer/soulmeasurer.kicad_pcb (KiCad board)
At the start: 2 copper layers, 40 x 46 mm, 28 parts, among them J1 OUTPUT, J2 INPUT, J3 LDO_GND, J4 LDO_VCC, J5 COMM, Q1 AP2055K, U1 INA229-Q1, U2 INA229-Q1, U3 AMS1117/WL9005P3

Commit message: Add panel
Routing:
- net SCLK: track 3.90 -> 15.3 mm, vias 1 -> 2
- net GND: vias 342 -> 344

Commit message: Rev 1: typo fixes
Parts:
- moved R4 0.75 mm to (111.8, 92.5), turned to 90 degrees
Connections:
- R4 pad 2: VBUS1 -> Net-(J1-Pin_1)
Routing:
- net Net-(J1-Pin_1): track 9.53 -> 17.3 mm
- net VBUS1: track 23.2 -> 19.7 mm, vias 0 -> 2
- net IN2+: track 5.98 -> 6.64 mm
- net GND: vias 344 -> 347
