File: soulmeasurer/soulmeasurer.kicad_sch (KiCad schematic)
At the start: 26 parts, among them J2 OUTPUT, J3 INPUT, J4 LDO_GND, J5 LDO_VCC, J5 MAIN_BOARD, Q1 AP2055K, U2 AMS1117/WL9005P3

Commit message: Finalise rev 1.0
Parts:
- removed J5: MAIN_BOARD, symbol Connector_Generic:Conn_02x06_Counter_Clockwise
- removed R1 (x2): 10k, Resistor_SMD:R_0603_1608Metric_Pad0.98x0.95mm_HandSolder, symbol Device:R
- added C9: 220uF, Capacitor_SMD:CP_Elec_10x12.6, symbol Device:C_Polarized
- added H1, H2, H3: M3_Hole, MountingHole:MountingHole_2.2mm_M2_ISO7380_Pad_TopBottom, symbol Mechanical:MountingHole_Pad
- added J5: COMM, Connector_PinSocket_2.54mm:PinSocket_2x07_P2.54mm_Vertical_SMD, symbol Connector_Generic:Conn_02x07_Odd_Even
- C1, C2: footprint (none) -> Capacitor_SMD:C_0603_1608Metric_Pad1.08x0.95mm_HandSolder
- C2: value 100nF -> 0.1uF
- R7: renamed from R9; footprint (none) -> Resistor_SMD:R_0603_1608Metric_Pad0.98x0.95mm_HandSolder
- U1, U2: value ~ -> INA229-Q1; footprint (none) -> Package_SO:VSSOP-10_3x3mm_P0.5mm
Connections:
- net +3V3: now also J5.6 (Pin_6), J5.8 (Pin_8)
- net +5V: now also J5.2 (Pin_2), J5.4 (Pin_4)
- net CS1: now also J5.1 (Pin_1)
- net CS2: now also J5.3 (Pin_3)
- net GND: now also U1.7 (GND), U2.7 (GND), H1.1, H2.1, H3.1, J5.13 (Pin_13), J5.14 (Pin_14)
- net HI_CURR_BYPASS: now also J5.10 (Pin_10)
- net MISO: now also J5.5 (Pin_5)
- net MOSI: now also J5.7 (Pin_7)
- net SCLK: now also J5.9 (Pin_9)
- net at J2.2 (Pin_2), J3.1 (Pin_1), J4.2 (Pin_2): now also C9.2
- net VBUS2: now reaches J3.2 (Pin_2), J5.1 (Pin_1), R2.1, R4.2
- net VBUS2: now also Q1.2 (D), U2.8 (VBUS), C9.1; no longer Q1.3 (S)
- net ALERT2: now reaches U2.3 (ALERT)
- net ALERT2: now also J5.12 (Pin_12)
- net VBUS1: now reaches R2.1, R2.2, R3.2, R4.2
- net VBUS1: now also Q1.3 (S), U1.8 (VBUS); no longer Q1.2 (D)
- net ALERT1: now reaches U1.3 (ALERT)
- net ALERT1: now also J5.11 (Pin_11)
- net VBUS: no longer names the net of J2.1 (Pin_1), R2.2, R3.2
- net VBUS: no longer U1.8 (VBUS), U2.8 (VBUS)
Other:
- moved on the sheet: J3, Q1, R7

Commit message: Rev 1: typo fixes
Connections:
- net VBUS1: no longer R3.2
- net at J2.1 (Pin_1), R2.2, R3.2: now also R3.2
Other:
- moved on the sheet: C2, R3, R4
